Commit message: Launchfile created - Folders models and worlds created

File: urdf/barista_robot_model.urdf (robot description, URDF)
Before this commit: robot urdfbot, 6 links, 5 joints
Links:
- added link back_caster_wheel; visual sphere radius=0.010
- added link front_caster_wheel; visual sphere radius=0.010
- link left_wheel: geometry visual cylinder length=0.0206 radius=0.0352
- link right_wheel: geometry visual cylinder length=0.0206 radius=0.0352
Joints:
- added joint base_link_to_back_caster_wheel_joint: type fixed, parent base_link, child back_caster_wheel, origin xyz=0 0 0 rpy=0 0 0
- added joint base_link_to_front_caster_wheel_joint: type fixed, parent base_link, child front_caster_wheel, origin xyz=0 0 0 rpy=0 0 0

Commit message: URDF file fixed - CMakelist fixed: Add config file to install

File: urdf/barista_robot_model.urdf (robot description, URDF)
Before this commit: robot urdfbot, 8 links, 7 joints
Links:
- removed link back_caster_wheel
- removed link front_caster_wheel
- added link back_pitch_link, mass 0.001; collision sphere radius=0.0352; visual sphere radius=0.0352
- added link back_roll_link, mass 0.001; collision cylinder length=0.001 radius=0.0352; visual cylinder length=0.001 radius=0.0352
- added link back_yaw_link, mass 0.001; collision cylinder length=0.001 radius=0.0352; visual cylinder length=0.001 radius=0.0352
- added link front_pitch_link, mass 0.001; collision sphere radius=0.0352; visual sphere radius=0.0352
- added link front_roll_link, mass 0.001; collision cylinder length=0.001 radius=0.0352; visual cylinder length=0.001 radius=0.0352
- added link front_yaw_link, mass 0.001; collision cylinder length=0.001 radius=0.0352; visual cylinder length=0.001 radius=0.0352
- added link laser_scan_frame
- added link laser_scan_link, mass 0.01; collision box size=0.02 0.02 0.02; visual box size=0.02 0.02 0.02
- added link laser_scan_model_link, mass 0.01; collision cylinder length=0.0408 radius=0.037493; visual mesh filename=package://barista_robot_description/meshes/sick_s300.dae scale=1.0 1.0 1.0
- link base_link: mass None -> 1.0; geometry collision cylinder length=0.155 radius=0.178; visual cylinder length=0.155 radius=0.178
- link cup_holder_tray: mass None -> 0.5; geometry collision cylinder length=0.09 radius=0.16; visual cylinder length=0.09 radius=0.16
- link left_wheel: mass None -> 0.1; geometry collision cylinder length=0.0206 radius=0.0352; visual cylinder length=0.0206 radius=0.0352
- link right_wheel: mass None -> 0.1; geometry collision cylinder length=0.0206 radius=0.0352; visual cylinder length=0.0206 radius=0.0352
- link standoff_rods_1: mass None -> 0.1; geometry collision cylinder length=0.22 radius=0.01; visual cylinder length=0.22 radius=0.01
- link standoff_rods_2: mass None -> 0.1; geometry collision cylinder length=0.22 radius=0.01; visual cylinder length=0.22 radius=0.01
Joints:
- removed joint base_link_to_back_caster_wheel_joint
- removed joint base_link_to_front_caster_wheel_joint
- removed joint standoff_rods_1_to_cup_holder_tray_joint
- added joint back_pitch_joint: type continuous, parent back_roll_link, child back_pitch_link, origin xyz=0 0 0 rpy=0 0 0, axis 0 1 0, limit effort=1000.0 velocity=100.0
- added joint back_roll_joint: type continuous, parent back_yaw_link, child back_roll_link, origin xyz=0 0 0 rpy=0 0 0, axis 1 0 0, limit effort=1000.0 velocity=100.0
- added joint back_yaw_joint: type continuous, parent base_link, child back_yaw_link, origin xyz=0 -0.1 -0.0775 rpy=0 0 0, axis 0 0 1, limit effort=1000.0 velocity=100.0
- added joint base_link_to_cup_holder_tray_joint: type fixed, parent base_link, child cup_holder_tray, origin xyz=0 0 0.3425 rpy=0 0 0
- added joint front_pitch_joint: type continuous, parent front_roll_link, child front_pitch_link, origin xyz=0 0 0 rpy=0 0 0, axis 0 1 0, limit effort=1000.0 velocity=100.0
- added joint front_roll_joint: type continuous, parent front_yaw_link, child front_roll_link, origin xyz=0 0 0 rpy=0 0 0, axis 1 0 0, limit effort=1000.0 velocity=100.0
- added joint front_yaw_joint: type continuous, parent base_link, child front_yaw_link, origin xyz=0 0.1 -0.0775 rpy=0 0 0, axis 0 0 1, limit effort=1000.0 velocity=100.0
- added joint laser_scan_frame_joint: type fixed, parent laser_scan_link, child laser_scan_frame, origin xyz=0 0 0.03 rpy=0 0 0, axis 0 0 0
- added joint laser_scan_link_joint: type prismatic, parent base_link, child laser_scan_link, origin xyz=0.0 0.0 0.155 rpy=0 0 0, axis 0 0 1, limit lower=-0.1 upper=0.0 effort=20.0 velocity=2.0
- added joint laser_scan_model_link_joint: type continuous, parent laser_scan_link, child laser_scan_model_link, origin xyz=0.0 0.0 0.0 rpy=0 0 0, axis 0 0 1, limit effort=10.0 velocity=2.0
- joint base_link_to_left_wheel_joint: axis (none) -> 1 0 0; limit (none) -> effort=10000 velocity=1000; origin xyz=0 0 0 rpy=0 0 0 -> xyz=0.11 0 -0.0775 rpy=0 0 0; type fixed -> continuous
- joint base_link_to_right_wheel_joint: axis (none) -> 1 0 0; limit (none) -> effort=10000 velocity=1000; origin xyz=0 0 0 rpy=0 0 0 -> xyz=-0.11 0 -0.0775 rpy=0 0 0; type fixed -> continuous
- joint base_link_to_standoff_rods_1_joint: origin xyz=0 0 0 rpy=0 0 0 -> xyz=0.10 0 0.1875 rpy=0 0 0
- joint base_link_to_standoff_rods_2_joint: origin xyz=0 0 0 rpy=0 0 0 -> xyz=-0.10 0 0.1875 rpy=0 0 0

Commit message: Colors in Gazebo match with colors in rviz - Two standoff rods added - LaserScan rays now appear in Gazebo - LaserScan rays position corrected

File: urdf/barista_robot_model.urdf (robot description, URDF)
Before this commit: robot barista_robot, 15 links, 14 joints
Links:
- added link standoff_rods_3, mass 0.1; collision cylinder length=0.22 radius=0.01; visual cylinder length=0.22 radius=0.01
- added link standoff_rods_4, mass 0.1; collision cylinder length=0.22 radius=0.01; visual cylinder length=0.22 radius=0.01
Joints:
- added joint base_link_to_standoff_rods_3_joint: type fixed, parent base_link, child standoff_rods_3, origin xyz=0.10 -0.05 0.1875 rpy=0 0 0
- added joint base_link_to_standoff_rods_4_joint: type fixed, parent base_link, child standoff_rods_4, origin xyz=-0.10 -0.05 0.1875 rpy=0 0 0
- joint base_link_to_standoff_rods_1_joint: origin xyz=0.10 0 0.1875 rpy=0 0 0 -> xyz=0.10 0.05 0.1875 rpy=0 0 0
- joint base_link_to_standoff_rods_2_joint: origin xyz=-0.10 0 0.1875 rpy=0 0 0 -> xyz=-0.10 0.05 0.1875 rpy=0 0 0
- joint laser_scan_link_joint: origin xyz=0.0 0.0 0.155 rpy=0 0 0 -> xyz=0.0 0.0 0.3 rpy=0 0 0
- joint laser_scan_model_link_joint: origin xyz=0.0 0.0 0.0 rpy=0 0 0 -> xyz=0.0 0.0 -0.145 rpy=0 0 -1.57

File: xacro/barista_robot_model.urdf.xacro (robot description, xacro)
@@ -17,4 +17,7 @@
         <color rgba="0.0 0.0 1.0 1"/>
     </material>
+    <material name="yellow">
+        <color rgba="1.0 1.0 0.0 1"/>
+    </material>
     <!-- ******************************************** Links ******************************************** -->
     <link name="base_link">
@@ -42,4 +45,6 @@
     <xacro:standoff standoff_name="standoff_rods_1"/>
     <xacro:standoff standoff_name="standoff_rods_2"/>
+    <xacro:standoff standoff_name="standoff_rods_3"/>
+    <xacro:standoff standoff_name="standoff_rods_4"/>
     <xacro:cup_holder_tray cup_holder_tray_name="cup_holder_tray"/>
     <gazebo reference="cup_holder_tray">
@@ -117,5 +122,5 @@
                 <sphere radius="0.0352"/>
             </geometry>
-            <material name="green_dark"/>
+            <material name="yellow"/>
         </visual>
         <collision>
@@ -136,5 +141,5 @@
         <mu1>0.5</mu1>
         <mu2>0.5</mu2>
-        <material>Gazebo/Purple</material>
+        <material>Gazebo/Yellow</material>
     </gazebo>
     <!-- Caster Wheel Back -->
@@ -191,5 +196,5 @@
             <sphere radius="0.0352"/>
             </geometry>
-            <material name="green_light"/>
+            <material name="yellow"/>
         </visual>
         <collision>
@@ -256,5 +261,6 @@
             <!-- Laser Position Control-->
             <joint name="laser_scan_link_joint" type="prismatic">
-                <origin rpy="0 0 0" xyz="0.0 0.0 0.155"/>
+                <!--origin rpy="0 0 0" xyz="0.0 0.0 0.155"/-->
+                <origin rpy="0 0 0" xyz="0.0 0.0 0.3"/>
                 <parent link="base_link"/>
                 <child link="laser_scan_link"/>
@@ -263,6 +269,7 @@
                 <dynamics damping="0.1" friction="1.0"/>
             </joint>
+            <!-- -->>
             <joint name="laser_scan_frame_joint" type="fixed">
-                <origin rpy="0 0 0" xyz="0 0 0.03"/>
+                <origin rpy="0 0 0" xyz="0 0 0.0"/>
                 <parent link="laser_scan_link"/>
                 <child link="laser_scan_frame"/>
@@ -271,5 +278,6 @@
             <!-- Visual Laser Model to be rotated -->
             <joint name="laser_scan_model_link_joint" type="continuous">
-                <origin rpy="0 0 0" xyz="0.0 0.0 0.0"/>
+                <!--origin rpy="0 0 -1.57" xyz="0.0 0.0 0.0"/-->
+                <origin rpy="0 0 -1.57" xyz="0.0 0.0 -0.145"/>
                 <parent link="laser_scan_link"/>
                 <child link="laser_scan_model_link"/>
@@ -336,12 +344,22 @@
     <!-- ******************************************** Joints ******************************************** -->
     <joint name="base_link_to_standoff_rods_1_joint" type="fixed">
-        <origin rpy="0 0 0" xyz="0.10 0 0.1875" />
+        <origin rpy="0 0 0" xyz="0.10 0.05 0.1875" />
         <parent link="base_link" />
         <child link="standoff_rods_1" />
     </joint>
     <joint name="base_link_to_standoff_rods_2_joint" type="fixed">
-        <origin rpy="0 0 0" xyz="-0.10 0 0.1875" />
+        <origin rpy="0 0 0" xyz="-0.10 0.05 0.1875" />
         <parent link="base_link" />
         <child link="standoff_rods_2" />
+    </joint>
+    <joint name="base_link_to_standoff_rods_3_joint" type="fixed">
+        <origin rpy="0 0 0" xyz="0.10 -0.05 0.1875" />
+        <parent link="base_link" />
+        <child link="standoff_rods_3" />
+    </joint>
+    <joint name="base_link_to_standoff_rods_4_joint" type="fixed">
+        <origin rpy="0 0 0" xyz="-0.10 -0.05 0.1875" />
+        <parent link="base_link" />
+        <child link="standoff_rods_4" />
     </joint>
     <joint name="base_link_to_cup_holder_tray_joint" type="fixed">

File: xacro/standoff.xacro (robot description, xacro)
@@ -3,4 +3,7 @@
     <xacro:property name="rod_length" value="0.22"/>
     <xacro:property name="rod_width" value="0.01"/>
+    <material name="white">
+        <color rgba="1.0 1.0 1.0 1"/>
+    </material>
     <xacro:macro name="standoff" params="standoff_name">
         <link name="${standoff_name}">
@@ -10,5 +13,5 @@
                     <cylinder length="${rod_length}" radius="${rod_width}"/>
                 </geometry>
-                <material name="red"/>
+                <material name="white"/>
             </visual>
             <collision>

File: xacro/wheel.xacro (robot description, xacro)
@@ -3,4 +3,7 @@
     <xacro:property name="wheel_radius" value="0.0352"/>
     <xacro:property name="wheel_width" value="0.0206"/>
+    <material name="black">
+        <color rgba="0.0 0.0 0.0 1"/>
+    </material>
     <xacro:macro name="wheel" params="wheel_name">
         <link name="${wheel_name}">
@@ -10,5 +13,5 @@
                     <cylinder length="${wheel_width}" radius="${wheel_radius}"/>
                 </geometry>
-                <material name="red"/>
+                <material name="black"/>
             </visual>
             <collision>
