Commit message: barista_two_robots launchfile added - Broadcaster for rick and morty robots added, scripts folder - xacro file modified to accept different robot names

File: xacro/barista_robot_model.urdf.xacro (robot description, xacro)
@@ -1,4 +1,5 @@
 <?xml version="1.0"?>
 <robot xmlns:xacro="http://www.ros.org/wiki/xacro" name="barista_robot">
+    <xacro:property name="robot_name" value="$(arg robot_name)"/>
     <xacro:property name="include_laser" default="true" />
     <xacro:include filename="$(find barista_robot_description)/xacro/wheel.xacro" />
@@ -308,4 +309,5 @@
                     <plugin name="laser" filename="libgazebo_ros_ray_sensor.so">
                     <ros>
+                        <namespace>/${robot_name}</namespace>
                         <remapping>~/out:=scan</remapping>
                     </ros>
@@ -437,4 +439,5 @@
         <plugin name="box_bot_joint_state" filename="libgazebo_ros_joint_state_publisher.so">
             <ros>
+                <namespace>/${robot_name}</namespace>
                 <remapping>~/out:=joint_states</remapping>
             </ros>
@@ -456,4 +459,8 @@
     <gazebo>
         <plugin filename="libgazebo_ros_diff_drive.so" name="differential_drive_controller">
+            <ros>
+                <namespace>/${robot_name}</namespace>
+                <remapping>/cmd_vel:=cmd_vel</remapping>
+            </ros>
             <!-- wheels -->
             <left_joint>base_link_to_left_wheel_joint</left_joint>
@@ -468,6 +475,6 @@
             <publish_odom>true</publish_odom>
             <publish_odom_tf>true</publish_odom_tf>
-            <odometry_frame>odom</odometry_frame>
-            <robot_base_frame>base_link</robot_base_frame>
+            <odometry_frame>${robot_name}/odom</odometry_frame>
+            <robot_base_frame>${robot_name}/base_link</robot_base_frame>
         </plugin>
     </gazebo>

Commit message: Base link fixed: now x-axis pointing to the front

File: xacro/barista_robot_model.urdf.xacro (robot description, xacro)
@@ -280,5 +280,5 @@
             <joint name="laser_scan_model_link_joint" type="continuous">
                 <!--origin rpy="0 0 -1.57" xyz="0.0 0.0 0.0"/-->
-                <origin rpy="0 0 -1.57" xyz="0.0 0.0 -0.145"/>
+                <origin rpy="0 0 0" xyz="0.0 0.0 -0.145"/>
                 <parent link="laser_scan_link"/>
                 <child link="laser_scan_model_link"/>
@@ -346,20 +346,20 @@
     <!-- ******************************************** Joints ******************************************** -->
     <joint name="base_link_to_standoff_rods_1_joint" type="fixed">
-        <origin rpy="0 0 0" xyz="0.10 0.05 0.1875" />
+        <origin rpy="0 0 0" xyz="0.05 0.10 0.1875" />
         <parent link="base_link" />
         <child link="standoff_rods_1" />
     </joint>
     <joint name="base_link_to_standoff_rods_2_joint" type="fixed">
-        <origin rpy="0 0 0" xyz="-0.10 0.05 0.1875" />
+        <origin rpy="0 0 0" xyz="-0.05 0.10 0.1875" />
         <parent link="base_link" />
         <child link="standoff_rods_2" />
     </joint>
     <joint name="base_link_to_standoff_rods_3_joint" type="fixed">
-        <origin rpy="0 0 0" xyz="0.10 -0.05 0.1875" />
+        <origin rpy="0 0 0" xyz="0.05 -0.10 0.1875" />
         <parent link="base_link" />
         <child link="standoff_rods_3" />
     </joint>
     <joint name="base_link_to_standoff_rods_4_joint" type="fixed">
-        <origin rpy="0 0 0" xyz="-0.10 -0.05 0.1875" />
+        <origin rpy="0 0 0" xyz="-0.05 -0.10 0.1875" />
         <parent link="base_link" />
         <child link="standoff_rods_4" />
@@ -371,21 +371,21 @@
     </joint>
     <joint name="base_link_to_left_wheel_joint" type="continuous">
-        <origin rpy="0 0 0" xyz="0.11 0 -0.0775" />
+        <origin rpy="0 0 0" xyz="0 0.11 -0.0775" />
         <parent link="base_link" />
         <child link="left_wheel" />
-        <axis rpy="0 0 0" xyz="1 0 0"/>
+        <axis rpy="0 0 0" xyz="0 1 0"/>
         <limit effort="10000" velocity="1000"/>
         <joint_properties damping="1.0" friction="1.0"/>
     </joint>
     <joint name="base_link_to_right_wheel_joint" type="continuous">
-        <origin rpy="0 0 0" xyz="-0.11 0 -0.0775" />
+        <origin rpy="0 0 0" xyz="0 -0.11 -0.0775" />
         <parent link="base_link" />
         <child link="right_wheel" />
-        <axis rpy="0 0 0" xyz="1 0 0"/>
+        <axis rpy="0 0 0" xyz="0 1 0"/>
         <limit effort="10000" velocity="1000"/>
         <joint_properties damping="1.0" friction="1.0"/>
     </joint>
     <joint name="front_yaw_joint" type="continuous">
-        <origin rpy="0 0 0" xyz="0 0.1 -0.0775"/>
+        <origin rpy="0 0 0" xyz="0.1 0 -0.0775"/>
         <parent link="base_link" />
         <child link="front_yaw_link" />
@@ -411,5 +411,5 @@
     </joint>
     <joint name="back_yaw_joint" type="continuous">
-        <origin rpy="0 0 0" xyz="0 -0.1 -0.0775"/>
+        <origin rpy="0 0 0" xyz="-0.1 0 -0.0775"/>
         <parent link="base_link" />
         <child link="back_yaw_link" />

File: xacro/wheel.xacro (robot description, xacro)
@@ -9,5 +9,5 @@
         <link name="${wheel_name}">
             <visual>
-                <origin rpy="0 1.5707 0" xyz="0 0 0"/>
+                <origin rpy="1.5707 0 0" xyz="0 0 0"/>
                 <geometry>
                     <cylinder length="${wheel_width}" radius="${wheel_radius}"/>
@@ -16,5 +16,5 @@
             </visual>
             <collision>
-                <origin rpy="0 1.5707 0" xyz="0 0 0"/>
+                <origin rpy="1.5707 0 0" xyz="0 0 0"/>
                 <geometry>
                     <cylinder length="${wheel_width}" radius="${wheel_radius}"/>

Commit message: Laser position and dimention fixed - Rick and Morty robots are now with different colors

File: xacro/barista_robot_model.urdf.xacro (robot description, xacro)
@@ -21,4 +21,15 @@
         <color rgba="1.0 1.0 0.0 1"/>
     </material>
+    <material name="black">
+        <color rgba="0.0 0.0 0.0 1"/>
+    </material>
+    <xacro:if value="${robot_name == 'rick'}">
+        <xacro:property name="body_color" default="blue" />
+        <xacro:property name="body_color_gazebo" default="Gazebo/Blue" />
+    </xacro:if>
+    <xacro:if value="${robot_name == 'morty'}">
+        <xacro:property name="body_color" default="red" />
+        <xacro:property name="body_color_gazebo" default="Gazebo/Red" />
+    </xacro:if>
     <!-- ******************************************** Links ******************************************** -->
     <link name="base_link">
@@ -28,5 +39,5 @@
                 <cylinder length="0.155" radius="0.178"/>
             </geometry>
-            <material name="red"/>
+            <material name="${body_color}"/>
         </visual>
         <collision>
@@ -42,5 +53,5 @@
     </link>
     <gazebo reference="base_link">
-        <material>Gazebo/Red</material>
+        <material>${body_color_gazebo}</material>
     </gazebo>
     <xacro:standoff standoff_name="standoff_rods_1"/>
@@ -48,7 +59,7 @@
     <xacro:standoff standoff_name="standoff_rods_3"/>
     <xacro:standoff standoff_name="standoff_rods_4"/>
-    <xacro:cup_holder_tray cup_holder_tray_name="cup_holder_tray"/>
+    <xacro:cup_holder_tray cup_holder_tray_name="cup_holder_tray" body_color="${body_color}"/>
     <gazebo reference="cup_holder_tray">
-        <material>Gazebo/Red</material>
+        <material>${body_color_gazebo}</material>
     </gazebo>
     <!-- Wheel Left -->
@@ -226,4 +237,5 @@
                         <box size="0.02 0.02 0.02"/>
                     </geometry>
+                    <material name="black"/>
                 </visual>
                 <collision>
@@ -245,11 +257,13 @@
                     <origin rpy="0 0 0" xyz="0 0 0"/>
                     <geometry>
-                        <mesh filename="package://barista_robot_description/meshes/sick_s300.dae" scale="1.0 1.0 1.0"/>
+                        <mesh filename="package://barista_robot_description/meshes/sick_s300.dae" scale="0.5 0.5 0.5"/>
                     </geometry>
+                    <material name="black"/>
                 </visual>
                 <collision>
                     <origin rpy="0 0 0" xyz="0 0 0.0204"/>
                     <geometry>
-                        <cylinder length="0.0408" radius="0.037493"/>
+                        <!--cylinder length="0.0408" radius="0.037493"/-->
+                        <mesh filename="package://barista_robot_description/meshes/sick_s300.dae" scale="0.5 0.5 0.5"/>
                     </geometry>
                 </collision>
@@ -262,6 +276,6 @@
             <!-- Laser Position Control-->
             <joint name="laser_scan_link_joint" type="prismatic">
-                <!--origin rpy="0 0 0" xyz="0.0 0.0 0.155"/-->
-                <origin rpy="0 0 0" xyz="0.0 0.0 0.3"/>
+                <origin rpy="0 0 0" xyz="0.0 0.0 0.175"/>
+                <!--origin rpy="0 0 0" xyz="0.0 0.0 0.2"/-->
                 <parent link="base_link"/>
                 <child link="laser_scan_link"/>
@@ -280,5 +294,5 @@
             <joint name="laser_scan_model_link_joint" type="continuous">
                 <!--origin rpy="0 0 -1.57" xyz="0.0 0.0 0.0"/-->
-                <origin rpy="0 0 0" xyz="0.0 0.0 -0.145"/>
+                <origin rpy="0 0 0" xyz="0.0 0.0 -0.055"/>
                 <parent link="laser_scan_link"/>
                 <child link="laser_scan_model_link"/>
@@ -340,4 +354,7 @@
                 </joint>
             </ros2_control>
+        <gazebo reference="laser_scan_model_link">
+            <material>Gazebo/Black</material>
+        </gazebo>
     </xacro:macro>
     <xacro:if value="${include_laser}">

File: xacro/cup_holder_tray.xacro (robot description, xacro)
@@ -1,5 +1,5 @@
 <?xml version="1.0"?>
 <robot xmlns:xacro="http://www.ros.org/wiki/xacro">
-    <xacro:macro name="cup_holder_tray" params="cup_holder_tray_name">
+    <xacro:macro name="cup_holder_tray" params="cup_holder_tray_name body_color">
         <link name="${cup_holder_tray_name}">
             <visual>
@@ -8,5 +8,5 @@
                     <cylinder length="0.09" radius="0.16"/>
                 </geometry>
-                <material name="red"/>
+                <material name="${body_color}"/>
             </visual>
             <collision>

File: xacro/wheel.xacro (robot description, xacro)
@@ -3,5 +3,5 @@
     <xacro:property name="wheel_radius" value="0.0352"/>
     <xacro:property name="wheel_width" value="0.0206"/>
-    <material name="black">
+    <material name="black_">
         <color rgba="0.0 0.0 0.0 1"/>
     </material>
@@ -13,5 +13,5 @@
                     <cylinder length="${wheel_width}" radius="${wheel_radius}"/>
                 </geometry>
-                <material name="black"/>
+                <material name="black_"/>
             </visual>
             <collision>
